File: LX1253/LX1253.kicad_pcb (KiCad board)
At the start: 2 copper layers, 37 parts, among them J1 Screw_Terminal_01x03, P1 SW_Push, U1 4017

Commit message: Prj spostato su gitlab
Parts:
- P1: footprint Button_Switch_SMD:SW_MEC_5GSH9 -> Button_Switch_THT:SW_PUSH_6mm_H4.3mm
- R1, R14, R15, R2: footprint Resistor_THT:R_Radial_Power_L13.0mm_W9.0mm_P5.00mm -> Resistor_THT:R_Axial_DIN0204_L3.6mm_D1.6mm_P7.62mm_Horizontal
- moved R1 178.2 mm to (61.2, 56.9), turned to 180 degrees
- moved C1 165.2 mm to (71.1, 101.4)
- moved OC1 163.5 mm to (219.7, 69.8)
- moved DL1 160.9 mm to (57.2, 88.4), turned to 180 degrees
- moved OC2 158.7 mm to (219.7, 109.2)
- moved R12 149.0 mm to (205.7, 101.6), turned to -90 degrees
- moved R15 145.4 mm to (212.1, 91.4), turned to 90 degrees
- moved C2 145.1 mm to (71.1, 37.6), turned to -90 degrees
- moved R2 132.1 mm to (82.8, 69.3), turned to 90 degrees
- moved R3 114.7 mm to (82.8, 93.2), turned to 90 degrees
- moved TR5 114.4 mm to (200.7, 87.6)
- moved R14 111.9 mm to (187.7, 57.9), turned to 0 degrees
- moved R13 110.5 mm to (199.4, 69.8)
- moved R4 98.9 mm to (92.7, 62.2), turned to -90 degrees
- moved R6 87.7 mm to (111.8, 50.8), turned to -90 degrees
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Routing:
- net GND: track 0.00 -> 345.8 mm
- net Net-(C4-Pad1): track 0.00 -> 216.8 mm
- net Net-(C1-Pad1): track 0.00 -> 161.4 mm
- net Net-(P1-Pad2): track 0.00 -> 87.0 mm
- net Net-(C3-Pad1): track 0.00 -> 59.9 mm
- net Net-(J1-Pad2): track 0.00 -> 57.7 mm
- net Net-(R8-Pad2): track 0.00 -> 56.2 mm
- net Net-(R4-Pad2): track 0.00 -> 53.0 mm
- net Net-(C2-Pad1): track 0.00 -> 45.2 mm
- net Net-(R10-Pad2): track 0.00 -> 34.8 mm
- net Net-(DL1-Pad2): track 0.00 -> 33.0 mm
- net Net-(OC1-Pad4): track 0.00 -> 32.3 mm
- net Net-(OC2-Pad2): track 0.00 -> 31.4 mm
- net Net-(R3-Pad2): track 0.00 -> 23.2 mm
- net Net-(C6-Pad1): track 0.00 -> 22.9 mm
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Other:
- board outline added: 202.7 x 85.9 mm
