File: LX1253/LX1253.kicad_sch (KiCad schematic)
At the start: 37 parts, among them J1 Screw_Terminal_01x03, P1 SW_Push, U1 4017

Commit message: Prj spostato su gitlab
Parts:
- C4: value (none) -> 100000 pF; footprint (none) -> Capacitor_THT:C_Rect_L10.0mm_W2.5mm_P7.50mm_MKS4
- P1: value SW_Push -> (none); footprint Button_Switch_SMD:SW_MEC_5GSH9 -> (none)
- R1, R14, R15, R2: footprint Resistor_THT:R_Radial_Power_L13.0mm_W9.0mm_P5.00mm -> Resistor_THT:R_Axial_DIN0204_L3.6mm_D1.6mm_P7.62mm_Horizontal
Changed lines of the file:
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@@
       (effects (font (size 1.27 1.27)) (justify right))
     )
-    (property "Value" "SW_Push" (id 1) (at 128.27 112.3949 90)
+    (property "Value" "" (id 1) (at 128.27 112.3949 90)
       (effects (font (size 1.27 1.27)) (justify right) hide)
     )
-    (property "Footprint" "Button_Switch_SMD:SW_MEC_5GSH9" (id 2) (at 121.92 111.125 0)
+    (property "Footprint" "" (id 2) (at 121.92 111.125 0)
       (effects (font (size 1.27 1.27)) hide)
     )
@@
       (effects (font (size 1.27 1.27)) (justify left) hide)
     )
-    (property "Footprint" "Resistor_THT:R_Radial_Power_L13.0mm_W9.0mm_P5.00mm" (id 2) (at 240.792 121.285 90)
+    (property "Footprint" "Resistor_THT:R_Axial_DIN0204_L3.6mm_D1.6mm_P7.62mm_Horizontal" (id 2) (at 240.792 121.285 90)
       (effects (font (size 1.27 1.27)) hide)
     )
@@
       (effects (font (size 1.27 1.27)) (justify left) hide)
     )
-    (property "Footprint" "Resistor_THT:R_Radial_Power_L13.0mm_W9.0mm_P5.00mm" (id 2) (at 240.792 51.435 90)
+    (property "Footprint" "Resistor_THT:R_Axial_DIN0204_L3.6mm_D1.6mm_P7.62mm_Horizontal" (id 2) (at 240.792 51.435 90)
       (effects (font (size 1.27 1.27)) hide)
     )
@@
       (effects (font (size 1.27 1.27)) hide)
     )
-    (property "Footprint" "Resistor_THT:R_Radial_Power_L13.0mm_W9.0mm_P5.00mm" (id 2) (at 69.215 39.243 90)
+    (property "Footprint" "Resistor_THT:R_Axial_DIN0204_L3.6mm_D1.6mm_P7.62mm_Horizontal" (id 2) (at 69.215 39.243 90)
       (effects (font (size 1.27 1.27)) hide)
     )
@@
       (effects (font (size 1.27 1.27)) (justify left) hide)
     )
-    (property "Footprint" "Resistor_THT:R_Radial_Power_L13.0mm_W9.0mm_P5.00mm" (id 2) (at 52.832 64.135 90)
+    (property "Footprint" "Resistor_THT:R_Axial_DIN0204_L3.6mm_D1.6mm_P7.62mm_Horizontal" (id 2) (at 52.832 64.135 90)
       (effects (font (size 1.27 1.27)) hide)
     )
@@
       (effects (font (size 1.27 1.27)) (justify left))
     )
-    (property "Value" "" (id 1) (at 156.21 42.5449 0)
-      (effects (font (size 1.27 1.27)) (justify left) hide)
-    )
-    (property "Footprint" "" (id 2) (at 153.3652 45.085 0)
+    (property "Value" "100000 pF" (id 1) (at 156.21 42.5449 0)
+      (effects (font (size 1.27 1.27)) (justify left) hide)
+    )
+    (property "Footprint" "Capacitor_THT:C_Rect_L10.0mm_W2.5mm_P7.50mm_MKS4" (id 2) (at 153.3652 45.085 0)
       (effects (font (size 1.27 1.27)) hide)
     )
@@
     )
     (path "/2bbd6c26-4114-4518-8f4a-c6fdadc046b6"
-      (reference "P1") (unit 1) (value "SW_Push") (footprint "Button_Switch_SMD:SW_MEC_5GSH9")
+      (reference "P1") (unit 1) (value "SW_Push") (footprint "Button_Switch_THT:SW_PUSH_6mm_H4.3mm")
     )
     (path "/d04eabf5-018b-4006-a739-ce16277681b7"
-      (reference "R1") (unit 1) (value "100") (footprint "Resistor_THT:R_Radial_Power_L13.0mm_W9.0mm_P5.00mm")
+      (reference "R1") (unit 1) (value "100") (footprint "Resistor_THT:R_Axial_DIN0204_L3.6mm_D1.6mm_P7.62mm_Horizontal")
     )
     (path "/b1240f00-ec43-4c0b-9a41-43264db8a893"
-      (reference "R2") (unit 1) (value "100") (footprint "Resistor_THT:R_Radial_Power_L13.0mm_W9.0mm_P5.00mm")
+      (reference "R2") (unit 1) (value "100") (footprint "Resistor_THT:R_Axial_DIN0204_L3.6mm_D1.6mm_P7.62mm_Horizontal")
     )
     (path "/54d76293-1ce2-46f8-9be7-a3d7f9f28112"
@@
     )
     (path "/9050328c-80d1-449f-94a8-27658961ba9d"
-      (reference "R14") (unit 1) (value "6800") (footprint "Resistor_THT:R_Radial_Power_L13.0mm_W9.0mm_P5.00mm")
+      (reference "R14") (unit 1) (value "6800") (footprint "Resistor_THT:R_Axial_DIN0204_L3.6mm_D1.6mm_P7.62mm_Horizontal")
     )
     (path "/7fd11519-eb9e-4413-8ca2-e43e38c699f6"
-      (reference "R15") (unit 1) (value "6800") (footprint "Resistor_THT:R_Radial_Power_L13.0mm_W9.0mm_P5.00mm")
+      (reference "R15") (unit 1) (value "6800") (footprint "Resistor_THT:R_Axial_DIN0204_L3.6mm_D1.6mm_P7.62mm_Horizontal")
     )
     (path "/6474aa6c-825c-4f0f-9938-759b68df02a5"
